File: HHC/2022/Circuits-Main.kicad_sch (KiCad schematic)
At the start: 0 parts

Commit message: Adding circuits workbook
Other:
- added sheet Capacitors (Circuits - Capacitors.kicad_sch)
- added sheet Circuit Symbols (Circuits - Symbols.kicad_sch)
- added sheet LEDs and Resistors (Circuits - LED Resistors.kicad_sch)
- added sheet Light the LED (Circuits - LED.kicad_sch)
- added sheet Reading Schematics (Circuits - Schematics.kicad_sch)
- added sheet Series and Parallel (Circuits - Series and Parallel.kicad_sch)
- added sheet The 555 - Astable (Circuits - 555 Astable.kicad_sch)
- added sheet The 555 - Monostable (Circuits - 555 Monostable.kicad_sch)
- company: (none) -> SAINTCON Hardware Hacking Community
- title: (none) -> Circuits Workbook - Main
Changed lines of the file:
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@@
 (kicad_sch (version 20211123) (generator eeschema)
-  (paper "A4")
+  (paper "USLetter")
+  (title_block
+    (title "Circuits Workbook - Main")
+    (date "2022-10-24")
+    (rev "1")
+    (company "SAINTCON Hardware Hacking Community")
+    (comment 1 "@hamster")
+  )
+  (sheet (at 31.496 144.526) (size 18.288 8.636) (fields_autoplaced)
+    (stroke (width 0.1524) (type solid) (color 0 0 0 0))
+    (fill (color 0 0 0 0.0000))
+    (property "Sheet name" "The 555 - Astable" (id 0) (at 31.496 143.8144 0)
+      (effects (font (size 1.27 1.27)) (justify left bottom))
+    )
+    (property "Sheet file" "Circuits - 555 Astable.kicad_sch" (id 1) (at 31.496 153.7466 0)
+      (effects (font (size 1.27 1.27)) (justify left top))
+    )
+  )
+  (sheet (at 31.496 123.444) (size 18.288 8.636) (fields_autoplaced)
+    (stroke (width 0.1524) (type solid) (color 0 0 0 0))
+    (fill (color 0 0 0 0.0000))
+    (property "Sheet name" "Capacitors" (id 0) (at 31.496 122.7324 0)
+      (effects (font (size 1.27 1.27)) (justify left bottom))
+    )
+    (property "Sheet file" "Circuits - Capacitors.kicad_sch" (id 1) (at 31.496 132.6646 0)
+      (effects (font (size 1.27 1.27)) (justify left top))
+    )
+  )
+  (sheet (at 31.496 25.908) (size 18.288 8.636) (fields_autoplaced)
+    (stroke (width 0.1524) (type solid) (color 0 0 0 0))
+    (fill (color 0 0 0 0.0000))
+    (property "Sheet name" "Circuit Symbols" (id 0) (at 31.496 25.1964 0)
+      (effects (font (size 1.27 1.27)) (justify left bottom))
+    )
+    (property "Sheet file" "Circuits - Symbols.kicad_sch" (id 1) (at 31.496 35.1286 0)
+      (effects (font (size 1.27 1.27)) (justify left top))
+    )
+  )
+  (sheet (at 31.75 67.564) (size 18.288 8.636) (fields_autoplaced)
+    (stroke (width 0.1524) (type solid) (color 0 0 0 0))
+    (fill (color 0 0 0 0.0000))
+    (property "Sheet name" "Light the LED" (id 0) (at 31.75 66.8524 0)
+      (effects (font (size 1.27 1.27)) (justify left bottom))
+    )
+    (property "Sheet file" "Circuits - LED.kicad_sch" (id 1) (at 31.75 76.7846 0)
+      (effects (font (size 1.27 1.27)) (justify left top))
+    )
+  )
+  (sheet (at 31.75 87.376) (size 18.288 8.636) (fields_autoplaced)
+    (stroke (width 0.1524) (type solid) (color 0 0 0 0))
+    (fill (color 0 0 0 0.0000))
+    (property "Sheet name" "LEDs and Resistors" (id 0) (at 31.75 86.6644 0)
+      (effects (font (size 1.27 1.27)) (justify left bottom))
+    )
+    (property "Sheet file" "Circuits - LED Resistors.kicad_sch" (id 1) (at 31.75 96.5966 0)
+      (effects (font (size 1.27 1.27)) (justify left top))
+    )
+  )
+  (sheet (at 31.496 165.862) (size 18.288 8.636) (fields_autoplaced)
+    (stroke (width 0.1524) (type solid) (color 0 0 0 0))
+    (fill (color 0 0 0 0.0000))
+    (property "Sheet name" "The 555 - Monostable" (id 0) (at 31.496 165.1504 0)
+      (effects (font (size 1.27 1.27)) (justify left bottom))
+    )
+    (property "Sheet file" "Circuits - 555 Monostable.kicad_sch" (id 1) (at 31.496 175.0826 0)
+      (effects (font (size 1.27 1.27)) (justify left top))
+    )
+  )
+  (sheet (at 31.496 46.99) (size 18.288 8.636) (fields_autoplaced)
+    (stroke (width 0.1524) (type solid) (color 0 0 0 0))
+    (fill (color 0 0 0 0.0000))
+    (property "Sheet name" "Reading Schematics" (id 0) (at 31.496 46.2784 0)
+      (effects (font (size 1.27 1.27)) (justify left bottom))
+    )
+    (property "Sheet file" "Circuits - Schematics.kicad_sch" (id 1) (at 31.496 56.2106 0)
+      (effects (font (size 1.27 1.27)) (justify left top))
+    )
+  )
+  (sheet (at 31.496 106.172) (size 18.288 8.636) (fields_autoplaced)
+    (stroke (width 0.1524) (type solid) (color 0 0 0 0))
+    (fill (color 0 0 0 0.0000))
+    (property "Sheet name" "Series and Parallel" (id 0) (at 31.496 105.4604 0)
+      (effects (font (size 1.27 1.27)) (justify left bottom))
+    )
+    (property "Sheet file" "Circuits - Series and Parallel.kicad_sch" (id 1) (at 31.496 115.3926 0)
+      (effects (font (size 1.27 1.27)) (justify left top))
+    )
+  )
 )
