File: HHC/2022/HHC-MiniBadge-2022.kicad_sch (KiCad schematic)
At the start: 48 parts, among them J1 Conn_01x02_Female, J10 Conn_01x01_Female, J11 Conn_01x01_Female, J12 Conn_01x01_Female, J13 Conn_01x01_Female, J14 Conn_01x01_Female, J15 Conn_01x01_Female, J16 Conn_01x01_Female, J17 Conn_01x01_Female, J18 Conn_01x01_Female, J19 Conn_01x01_Female, J2 Conn_01x02_Female, J20 Conn_01x01_Female, J21 Conn_01x01_Female, J22 Conn_01x01_Female, J23 Conn_01x01_Female, J24 Conn_01x01_Female, J25 Conn_01x01_Female, J26 Conn_01x01_Female, J27 Conn_01x01_Female, J28 Conn_01x02_Female, J29 Conn_01x02_Female, J3 Conn_01x02_Female, J4 Conn_01x02_Female, J5 Conn_01x02_Female, J6 Conn_01x01_Female, J7 Conn_01x01_Female, J8 Conn_01x01_Female, J9 Conn_01x01_Female, SW1 SW_Push, U1 NE555P, U2 SAINTCON-Minibadge, U3 SAINTCON-Minibadge, U4 SAINTCON-Minibadge, U5 SAINTCON-Minibadge

Commit message: Adding assembly guide
Other:
- added sheet Circut Workbook (Circuits-Main.kicad_sch)
Changed lines of the file:
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@@
     (pin "9")
+  )
+  (sheet (at 63.754 161.798) (size 24.13 13.462) (fields_autoplaced)
+    (stroke (width 0.1524) (type solid) (color 0 0 0 0))
+    (fill (color 0 0 0 0.0000))
+    (property "Sheet name" "Circut Workbook" (id 0) (at 63.754 161.0864 0)
+      (effects (font (size 1.27 1.27)) (justify left bottom))
+    )
+    (property "Sheet file" "Circuits-Main.kicad_sch" (id 1) (at 63.754 175.8446 0)
+      (effects (font (size 1.27 1.27)) (justify left top))
+    )
   )
   (sheet_instances
     (path "/" (page "1"))
+    (path "/26560972-4362-4887-bc88-50c3464405a4" (page "2"))
   )
   (symbol_instances

Commit message: Adding circuits workbook
Other:
- sheet Circut Workbook renamed Circuit Workbook
