File: HHC/2023/chc.kicad_pcb (KiCad board)
At the start: 2 copper layers, 20 x 20 mm, 12 parts

Commit message: Added panel for the 2023 minibadge
Parts:
- moved C1 39.3 mm to (153.4, 93.9)
- moved D1 39.3 mm to (136.9, 88.8)
- moved G*** 39.3 mm to (144.6, 96.9)
- moved MB1 39.3 mm to (134.5, 85.1)
- moved TP1 39.3 mm to (140.7, 88.7)
- moved TP2 39.3 mm to (148.3, 88.7)
- moved D2 39.3 mm to (152.5, 88.8)
- moved G*** 39.3 mm to (144.6, 96.8) (x2)
- moved R1 39.3 mm to (136.9, 91.0)
- moved R2 39.3 mm to (151.5, 93.7)
- moved R3 39.3 mm to (152.5, 91.0)
Other:
- board text added: "+3v3"
- board text added: "2023"
- board text added: "CLK"
- board text added: "GND"
- board text added: "SAINTCON CHC"
- board text added: "SQUARE"
- board text added: "TRIANGLE"
- board text added: "VBATT"
- board text added: "github.com/hamster/ saintcon"
- board text removed: "CHC 2023"
- board text removed: "github.com hamster/saintcon"
