File: Bitstream Hackers/2026/bhc.kicad_sch (KiCad schematic)
At the start: 7 parts, among them U1 AT24CS01-SSHM

Commit message: Adding finals, gerbers
Connections:
- net GND: now also MB1.8 (GND)
Other:
- moved on the sheet: D1, JP1, JP2, JP3, MB1, R1

Commit message: Small update on schematic graphics
Parts:
- R1: value 1k -> 33R
- U1: value AT24CS01-SSHM -> M24C08
Connections:
- no-connect marks 0 -> 7
Changed lines of the file:
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@@
 		(color 0 0 0 0)
+	)
+	(no_connect
+		(at 157.48 53.34)
+	)
+	(no_connect
+		(at 168.91 102.87)
+	)
+	(no_connect
+		(at 162.56 76.2)
+	)
+	(no_connect
+		(at 152.4 53.34)
+	)
+	(no_connect
+		(at 160.02 53.34)
+	)
+	(no_connect
+		(at 147.32 53.34)
+	)
+	(no_connect
+		(at 154.94 53.34)
 	)
 	(wire
@@
 		(fields_autoplaced yes)
 		(property "Reference" "R1"
-			(at 149.352 85.0899 0)
+			(at 149.86 85.0899 0)
 			(show_name no)
 			(do_not_autoplace no)
@@
 			)
 		)
-		(property "Value" "1k"
-			(at 149.352 87.6299 0)
+		(property "Value" "33R"
+			(at 149.86 87.6299 0)
 			(show_name no)
 			(do_not_autoplace no)
@@
 			)
 		)
-		(property "Value" "AT24CS01-SSHM"
-			(at 197.104 93.472 0)
-			(show_name no)
-			(do_not_autoplace no)
+		(property "Value" "M24C08"
+			(at 187.706 93.726 0)
+			(show_name no)
+			(do_not_autoplace no)
